File: hardware/SMD/mbanzi/AudioMega Oliver v101.sch (EAGLE design)
At the start: 72 parts, among them Q1 BC846ASMD, Q2 BC846ASMD, Q3 BC846ASMD, Q4 2N7002, Q5 BC846ASMD, Q6 BC846ASMD, U1 REG1117-5, U2 REG1117-3.3, U3 ATMEGA328-AU, U4 LM386M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

Commit message: Added Eagle 6.3.0 files for all my versions of the designs
Parts:
- removed C13: 100nF, resistor:C-USC1206
- removed C6: 10uF, resistor:C-USC1206
- removed Q6: BC846ASMD, transistor-npn:BC846ASMD
- removed R18: 2k2, resistor:R-US_R1206
- removed R19: 470, resistor:R-US_R1206
- removed R20, R21: 10k, resistor:R-US_R1206
- added C4: 10uF, resistor:CPOL-USCT3528
- added D4: BAT42, diode:DIODE-SOD123
- added JN1: 0, resistor:R-US_R1206
- C1, C3: device resistor:C-USC1206 -> resistor:CPOL-USCT3528
- C10, C16, C9: device resistor:C-USC1206 -> resistor:CPOL-USCT6032
- C18: value 10nF -> 4n7
- C20: value 47nF -> 22nF
- J1: device pinhead:PINHD-1X8 -> pinhead:PINHD-1X7
- JP13: value PD3 -> RXD-TTL5v
- JP15: value RXD -> PD3
- JP16: value TXD -> TXD-TTL5v
- JP3: value +5V -> BL+ (+5v)
- JP4: value BL -> BL-
- Q5: value BC846ASMD -> 2N7002; device transistor-npn:BC846ASMD -> zetex:NMOSSOT23; OC_FARNELL (none) -> unknown; OC_NEWARK (none) -> unknown
- R17: value 22k -> 1k
Connections:
- removed net N$14: C13.1, U4.BYPASS
- removed net N$40: D3.C, Q6.B, R20.1, R21.2
- removed net N$43: Q5.C, R18.2, R19.2
- removed net N$44: Q5.B, R17.2
- new net N$2: D4.A, Q5.S
- new net N$22: JN1.1, R17.1
- net +3V3: now also C4.+, Q5.G; no longer C6.1
- net +5V: now also C3.+, JN1.2; no longer C3.1, R18.1
- net GND: now also C1.-, C3.-, C4.-; no longer C1.2, C13.2, C3.2, C6.2, D3.A, Q5.E, Q6.E, R20.2
- net N$15: now also C10.-, C16.-, C9.-; no longer C10.1, C16.1, C9.1
- net N$17: now also C10.+, C16.+, C9.+; no longer C10.2, C16.2, C9.2
- net N$32: now also C1.+; no longer C1.1
- net N$37: now also D3.C; no longer R21.1
- net N$38: now also Q5.D; no longer R19.1
- net N$41: now also R17.2
- net N$42: now also D3.A; no longer Q6.C
- net N$46: now also D4.C; no longer R17.1
Other:
- note added: "'328 RX"
- note added: "'328 TX"
- moved on the sheet: C11, C12, C15, C17, C18, C19, C2, C20, C21, C22, C5, C8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
