File: hardware/SMD/mbanzi/9xVoice MikeB SMD v1_0b.brd (EAGLE design)
At the start: 78.1 x 45.5 mm, 83 parts, among them IC1 ATMEGA328P, IC2 LE33CZ, IC3 LM386M, IC4 REG1117, Q1 12MHz, T1 2N7002, T2 2N7002

Commit message: Added latest MikeB changes
Parts:
- removed D2: BAT81V, diode:SOD123
- removed DB0, DB1, DB2, DB3, LRXD, LTXD, MRD, MTD, RXD, TXD, X1, X2, X3: (no value), pinhead:1X01
- removed T1: 2N7002, zetex:SOT-23
- removed U$1: (no value), SparkFun-Aesthetics:OSHW-LOGO-M
- added D0123: (no value), jdc:1X04
- added LTRXD, MTRD, TRXD: (no value), jdc:1X02
- added R24: 10K, rcl:R1206
- added X123: (no value), jdc:1X03
- C13: value 330p -> 470p
- C18: value 0.0047u -> 3900p
- C19: value 0.022u -> 10000p
- moved S1 30.9 mm to (16.0, 10.8)
- moved Q1 4.81 mm to (32.8, 24.8), turned to 225 degrees
- moved C19 4.26 mm to (30.8, 31.5), turned to 90 degrees
- moved GND 2.50 mm to (25.2, 39.8)
- moved C8 1.66 mm to (33.8, 31.5), turned to 90 degrees
- moved SUPPLY 1.00 mm to (25.2, 42.2)
- moved SGND 0.50 mm to (75.8, 16.5)
- moved C7 0.06 mm to (39.5, 31.5)
Connections:
- net N$24 renamed BEEPER
- removed net N$12: D4.C, LRXD.1
- removed net N$15: D2.A, T1.2
- removed net N$16: MTD.1, T1.1
- removed net N$17: LTXD.1, T2.1
- removed net N$18: D1.C, MRD.1
- removed net N$38: C13.1, IC3.3, R13.2, R23.1
- removed net N$7: IC1.26, X1.1
- removed net N$8: IC1.25, X2.1
- removed net N$9: IC1.24, X3.1
- removed net TXD: D2.C, D5.C, IC1.31, R20.2
- new net LRXD: D4.C, LTRXD.2
- new net LTXD: LTRXD.1, T2.1
- new net MRD: D1.C, MTRD.2
- new net MTD: D5.C, IC1.31, MTRD.1, R20.2, R24.1
- new net N$1: C13.1, R13.2, R23.1
- new net X1: IC1.26, X123.1
- new net X2: IC1.25, X123.2
- new net X3: IC1.24, X123.3
- net 3V3: no longer T1.3
- net 5V: now also R24.2
- net LCD_D0: now also D0123.1; no longer DB0.1
- net LCD_D1: now also D0123.2; no longer DB1.1
- net LCD_D2: now also D0123.3; no longer DB2.1
- net LCD_D3: now also D0123.4; no longer DB3.1
- net N$10: now also TRXD.2; no longer RXD.1
- net N$3: now also TRXD.1; no longer TXD.1
- net N$40: now also IC3.3
Routing:
- net MTD: track 0.00 -> 67.6 mm, vias 0 -> 2
- net TXD: track 55.2 -> 0.00 mm, vias 2 -> 0
- net 5V: track 72.2 -> 124.6 mm, vias 1 -> 2
- net BATTERY: track 22.1 -> 57.6 mm
- net X1: track 0.00 -> 27.3 mm
- net N$7: track 27.0 -> 0.00 mm
- net 3V3: track 118.0 -> 93.6 mm, vias 3 -> 2
- net X2: track 0.00 -> 20.6 mm
- net N$8: track 20.5 -> 0.00 mm
- net N$38: track 18.3 -> 0.00 mm, vias 2 -> 0
- net N$9: track 10.8 -> 0.00 mm
- net X3: track 0.00 -> 10.5 mm
- net MRD: track 0.00 -> 7.79 mm
- net N$18: track 7.27 -> 0.00 mm
- net N$1: track 0.00 -> 7.13 mm
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Other:
- board text added: "+5V"
- board text added: "+Ub"
- board text added: "C"
- board text added: "D0"
- board text added: "D1"
- board text added: "D2"
- board text added: "D3"
- board text added: "LRXD"
- board text added: "LTXD"
- board text added: "MRD"
- board text added: "MTD"
- board text added: "RXD"
- board text added: "TXD"
- board text added: "X1"
- board text added: "X2"
- board text added: "X3"
- board text added: "v1.0b"
- board text removed: "v1"
