File: hardware/SMD/mbanzi/9xVoice MikeB SMD v1_0b.sch (EAGLE design)
At the start: 82 parts, among them IC1 ATMEGA328P, IC2 LE33CZ, IC3 LM386M, IC4 REG1117, Q1 12MHz, T1 2N7002, T2 2N7002

Commit message: Added latest MikeB changes
Parts:
- removed D2: BAT81V, diode:DIODE-SOD123
- removed DB0, DB1, DB2, DB3, LRXD, LTXD, MRD, MTD, RXD, TXD, X1, X2, X3: (no value), pinhead:PINHD-1X1
- removed T1: 2N7002, zetex:NMOSSOT23
- added D0123: (no value), jdc:PINHD-1X4
- added LTRXD, MTRD, TRXD: (no value), jdc:PINHD-1X2
- added R24: 10K, rcl:R-US_R1206
- added X123: (no value), jdc:PINHD-1X3
- C13: value 330p -> 470p
- C18: value 0.0047u -> 3900p
- C19: value 0.022u -> 10000p
Connections:
- net N$24 renamed BEEPER
- removed net N$12: D4.C, LRXD.1
- removed net N$15: D2.A, T1.S
- removed net N$16: MTD.1, T1.D
- removed net N$17: LTXD.1, T2.D
- removed net N$18: D1.C, MRD.1
- removed net N$38: C13.1, IC3.+IN, R13.2, R23.1
- removed net N$7: IC1.PC3(ADC3), X1.1
- removed net N$8: IC1.PC2(ADC2), X2.1
- removed net N$9: IC1.PC1(ADC1), X3.1
- removed net TXD: D2.C, D5.C, IC1.PD1(TXD), R20.2
- new net LRXD: D4.C, LTRXD.2
- new net LTXD: LTRXD.1, T2.D
- new net MRD: D1.C, MTRD.2
- new net MTD: D5.C, IC1.PD1(TXD), MTRD.1, R20.2, R24.1
- new net N$1: C13.1, R13.2, R23.1
- new net X1: IC1.PC3(ADC3), X123.1
- new net X2: IC1.PC2(ADC2), X123.2
- new net X3: IC1.PC1(ADC1), X123.3
- net 3V3: no longer T1.G
- net 5V: now also R24.2
- net LCD_D0: now also D0123.1; no longer DB0.1
- net LCD_D1: now also D0123.2; no longer DB1.1
- net LCD_D2: now also D0123.3; no longer DB2.1
- net LCD_D3: now also D0123.4; no longer DB3.1
- net N$10: now also TRXD.2; no longer RXD.1
- net N$3: now also TRXD.1; no longer TXD.1
- net N$40: now also IC3.+IN
