File: hardware/SMD/Oliver/v102/AudioMega v102.sch (EAGLE design)
At the start: 74 parts, among them Q1 BC846ASMD, Q2 BC846ASMD, Q3 BC846ASMD, Q4 2N7002, Q5 BC846ASMD, U1 REG1117-5, U2 REG1117-3.3, U3 ATMEGA328-AU, U4 LM386M, X1 12MHz

Commit message: updated v102 board + added connector for haptic motor + added last schematic changes from MikeB (connection to M64) + added last audio filter changes (filtering PWM noise) from Mike and Hans
Parts:
- removed JN1, JN2: 0, resistor:R-US_R1206
- added C6: 330pf, resistor:C-USC1206
- added R20: 47k, resistor:R-US_R1206
- R9: value 33k -> 47k
Connections:
- removed net N$14: U4.BYPASS
- removed net N$22: JN2.1, R17.1
- removed net N$44: JP20.1, Q5.C
- new net N$61: C8.1, R20.2
- net +5V: now also Q5.C; no longer JP19.1
- net GND: now also C6.2, JP20.1; no longer Q5.E
- net N$2: now also JP19.1, Q5.E; no longer JN1.2, JN2.2, JP15.1
- net N$24: now also C6.1, R20.1; no longer C8.1
- net N$38: now also JP15.1, R17.1; no longer JN1.1
Other:
- moved on the sheet: C18, JP18, JP19, JP20, Q5, R10, R14, R18, R19, R9

Commit message: updated v102 board - checked for Gerber export - add Gerber files
Parts:
- renumbered JP1 to UB+, JP10 to SP+, JP11 to SP-, JP12 to PD2, JP13 to TX, JP14 to BEP, JP15 to PD3, JP16 to RX, JP17 to GND, JP18 to PG2, JP19 to HAP+, JP2 to UGND, JP20 to HAPG, JP3 to BL+, JP4 to BL-, JP5 to PB7, JP6 to LCD0, JP7 to LCD1, JP8 to LCD2, JP9 to LCD3
